Commit message: add measurement data

File: src/mbot_sim/urdf/xacro/mbot.xacro (robot description, xacro)
@@ -2,7 +2,7 @@
     <xacro:include filename="$(find mbot_sim)/urdf/xacro/mbot_base.xacro" />
     <xacro:include filename="$(find mbot_sim)/urdf/xacro/mbot_camera.xacro" />
-    <xacro:property name="camera_offset_x" value="0.17" />
+    <xacro:property name="camera_offset_x" value="0.2" />
     <xacro:property name="camera_offset_y" value="0" />
-    <xacro:property name="camera_offset_z" value="0.10" />
+    <xacro:property name="camera_offset_z" value="0" />
     <xacro:mbot_base_gazebo/>
     <!-- Camera -->

File: src/mbot_sim/urdf/xacro/mbot_camera.xacro (robot description, xacro)
@@ -78,5 +78,5 @@
 		        <distortion_t1>0.0</distortion_t1>
 		        <distortion_t2>0.0</distortion_t2>
-                <pointCloudCutoff>0.4</pointCloudCutoff>
+                <pointCloudCutoff>0</pointCloudCutoff>
             </plugin>
             </sensor>
